File: ZVS-Driver_pcb/ZVS-Driver.kicad_pcb (KiCad board)
At the start: 2 copper layers, 163 x 96.2 mm, 25 parts, among them J1 Screw_Terminal_01x02, J3 Screw_Terminal_01x04, Q1 IRF540N, Q2 IRF540N, Q3 IRF540N, Q4 IRF540N, Q5 IRF540N

Commit message: Spiti alex
Connections:
- J3 pad 2: 0 -> unconnected-(J3-Pin_2-Pad2)
- J3 pad 3: Net-(D4-K) -> unconnected-(J3-Pin_3-Pad3)
- J3 pad 4: unconnected-(J3-Pin_4-Pad4) -> Net-(D4-K)
- L1 pad 1: Net-(D1-K) -> Net-(D6-K)
- L1 pad 2: Net-(D6-K) -> Net-(D1-K)
Routing:
- net Net-(D3-K): track 269.5 -> 250.8 mm
- net 0: track 322.2 -> 307.0 mm
- net Net-(D1-K): track 79.6 -> 65.3 mm
- net Net-(D4-K): track 301.6 -> 303.9 mm
- net Net-(D6-K): track 79.8 -> 78.1 mm
Changed lines of the file:
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@@
 	(net 7 "Net-(D4-K)")
 	(net 8 "Net-(Q3-D)")
-	(net 9 "unconnected-(J3-Pin_4-Pad4)")
+	(net 9 "unconnected-(J3-Pin_3-Pad3)")
+	(net 10 "unconnected-(J3-Pin_2-Pad2)")
 	(footprint "Diode_THT:D_DO-41_SOD81_P12.70mm_Horizontal"
 		(layer "F.Cu")
@@
 			(layers "*.Cu" "*.Mask")
 			(remove_unused_layers no)
-			(net 2 "Net-(D1-K)")
+			(net 1 "Net-(D6-K)")
 			(pinfunction "1")
 			(pintype "passive")
@@
 			(layers "*.Cu" "*.Mask")
 			(remove_unused_layers no)
-			(net 1 "Net-(D6-K)")
+			(net 2 "Net-(D1-K)")
 			(pinfunction "2")
 			(pintype "passive")
@@
 			)
 		)
-		(pad "2" thru_hole circle
+		(pad "1" thru_hole circle
 			(at 0 0 90)
 			(size 1.6 1.6)
@@
 			(remove_unused_layers no)
 			(net 3 "0")
-			(pinfunction "Pin_2")
+			(pinfunction "Pin_1")
 			(pintype "passive")
 		)
 		(pad "2" thru_hole circle
-			(at 7.62 0 90)
+			(at 2.54 0 90)
 			(size 1.6 1.6)
 			(drill 0.8)
 			(layers "*.Cu" "*.Mask")
 			(remove_unused_layers no)
-			(net 3 "0")
+			(net 10 "unconnected-(J3-Pin_2-Pad2)")
 			(pinfunction "Pin_2")
 			(pintype "passive")
 		)
 		(pad "3" thru_hole circle
-			(at 2.54 0 90)
+			(at 5.08 0 90)
 			(size 1.6 1.6)
 			(drill 0.8)
 			(layers "*.Cu" "*.Mask")
 			(remove_unused_layers no)
-			(net 7 "Net-(D4-K)")
+			(net 9 "unconnected-(J3-Pin_3-Pad3)")
 			(pinfunction "Pin_3")
 			(pintype "passive")
 		)
 		(pad "4" thru_hole circle
-			(at 5.08 0 90)
+			(at 7.62 0 90)
 			(size 1.6 1.6)
 			(drill 0.8)
 			(layers "*.Cu" "*.Mask")
 			(remove_unused_layers no)
-			(net 9 "unconnected-(J3-Pin_4-Pad4)")
+			(net 7 "Net-(D4-K)")
 			(pinfunction "Pin_4")
 			(pintype "passive")
@@
 			(keep_text_aligned yes)
 		)
-		(gr_text "12.5"
+		(gr_text "12,5"
 			(at 167.05 77.25 90)
 			(layer "User.1")
@@
 			(keep_text_aligned yes)
 		)
-		(gr_text "4.75"
+		(gr_text "4,75"
 			(at 110.05 62.125 90)
 			(layer "User.1")
@@
 			(keep_text_aligned yes)
 		)
-		(gr_text "4.75"
+		(gr_text "4,75"
 			(at 110.05 122.875 90)
 			(layer "User.1")
@@
 			(keep_text_aligned yes)
 		)
-		(gr_text "12.5"
+		(gr_text "12,5"
 			(at 168.55 108.25 90)
 			(layer "User.1")
@@
 	)
 	(segment
+		(start 163.3 100.4)
+		(end 169.499 94.201)
+		(width 4)
+		(layer "F.Cu")
+		(net 1)
+	)
+	(segment
 		(start 134.376 121.101)
 		(end 124.625 111.35)
@@
 		(start 159 100.4)
 		(end 163.3 100.4)
-		(width 1)
+		(width 4)
 		(layer "F.Cu")
 		(net 1)
 	)
 	(segment
-		(start 163.3 100.4)
-		(end 173.7 90)
+		(start 145.113156 121.101)
+		(end 134.376 121.101)
 		(width 1)
 		(layer "F.Cu")
@@
 	)
 	(segment
-		(start 145.113156 121.101)
-		(end 134.376 121.101)
-		(width 1)
+		(start 169.499 94.201)
+		(end 173.7 94.201)
+		(width 4)
 		(layer "F.Cu")
 		(net 1)
@@
 	)
 	(segment
-		(start 176 94)
-		(end 180 90)
+		(start 159 71.05)
+		(end 158.95 71)
 		(width 4)
 		(layer "F.Cu")
@@
 	)
 	(segment
-		(start 159 71.05)
-		(end 158.95 71)
+		(start 169.1 85.4)
+		(end 173.7 90)
 		(width 4)
 		(layer "F.Cu")
@@
 	)
 	(segment
-		(start 175.4 85.4)
-		(end 159 85.4)
-		(width 4)
-		(layer "F.Cu")
-		(net 2)
-	)
-	(segment
-		(start 180 90)
-		(end 175.4 85.4)
-		(width 4)
-		(layer "F.Cu")
-		(net 2)
-	)
-	(segment
-		(start 173.7 94)
-		(end 176 94)
+		(start 159 85.4)
+		(end 169.1 85.4)
 		(width 4)
 		(layer "F.Cu")
@@
 	)
 	(segment
-		(start 64.9 120.42)
-		(end 74.201 111.119)
-		(width 1)
-		(layer "B.Cu")
-		(net 3)
-	)
-	(segment
-		(start 73.321735 96.499)
-		(end 58.701 96.499)
-		(width 1)
+		(start 71.11 134.25)
+		(end 98.33 134.25)
+		(width 2)
 		(layer "B.Cu")
 		(net 3)
@@
 	)
 	(segment
-		(start 58.701 96.499)
-		(end 52.7 102.5)
-		(width 1)
-		(layer "B.Cu")
-		(net 3)
-	)
-	(segment
 		(start 93.25 95.65)
 		(end 93.25 113)
@@
 	)
 	(segment
-		(start 94.14 113.89)
-		(end 93.25 113)
-		(width 1)
+		(start 64.9 128.04)
+		(end 71.11 134.25)
+		(width 2)
 		(layer "B.Cu")
 		(net 3)
 	)
 	(segment
-		(start 74.201 97.378265)
-		(end 73.321735 96.499)
+		(start 94.14 113.89)
+		(end 93.25 113)
 		(width 1)
 		(layer "B.Cu")
@@
 	)
 	(segment
-		(start 74.201 111.119)
-		(end 74.201 97.378265)
-		(width 1)
-		(layer "B.Cu")
-		(net 3)
-	)
-	(segment
 		(start 45.23 94.5)
 		(end 52.78 86.95)
@@
 	)
 	(segment
-		(start 105.95 59.75)
-		(end 101.7 55.5)
+		(start 130 63)
+		(end 130 68.19)
 		(width 1)
 		(layer "F.Cu")
@@
 	)
 	(segment
-		(start 124.65 73.54)
-		(end 119.74 73.54)
+		(start 105.95 59.75)
+		(end 101.7 55.5)
 		(width 1)
 		(layer "F.Cu")
@@
 	)
 	(segment
-		(start 59.19 78)
-		(end 75 78)
+		(start 141 52)
+		(end 130 63)
 		(width 1)
 		(layer "F.Cu")
@@
 	)
 	(segment
-		(start 50.24 86.95)
-		(end 59.19 78)
+		(start 124.65 73.54)
+		(end 119.74 73.54)
 		(width 1)
 		(layer "F.Cu")
@@
 	)
 	(segment
-		(start 75 78)
-		(end 84.01 68.99)
+		(start 158.95 127.2)
+		(end 178 108.15)
 		(width 1)
 		(layer "F.Cu")
@@
 	)
 	(segment
-		(start 84.01 68.99)
-		(end 84.01 55.5)
+		(start 59.19 78)
+		(end 75 78)
 		(width 1)
 		(layer "F.Cu")
@@
 	)
 	(segment
-		(start 101.7 55.5)
-		(end 84.01 55.5)
+		(start 50.24 86.95)
+		(end 59.19 78)
 		(width 1)
 		(layer "F.Cu")
@@
 	)
 	(segment
-		(start 105.95 59.75)
-		(end 105.95 50.75)
+		(start 178 68)
+		(end 162 52)
 		(width 1)
 		(layer "F.Cu")
@@
 	)
 	(segment
-		(start 164 51)
-		(end 158 51)
-		(width 2)
-		(layer "B.Cu")
-		(net 6)
-	)
-	(segment
-		(start 158.95 127.2)
-		(end 175.701 110.449)
-		(width 2)
-		(layer "B.Cu")
-		(net 6)
-	)
-	(segment
-		(start 175.701 110.449)
-		(end 175.701 62.701)
-		(width 2)
-		(layer "B.Cu")
+		(start 130 68.19)
+		(end 124.65 73.54)
+		(width 1)
+		(layer "F.Cu")
 		(net 6)
 	)
 	(segment
-		(start 146 84)
-		(end 135.11 84)
-		(width 2)
-		(layer "B.Cu")
+		(start 162 52)
+		(end 141 52)
+		(width 1)
+		(layer "F.Cu")
 		(net 6)
 	)
 	(segment
-		(start 151 58)
-		(end 151 79)
-		(width 2)
-		(layer "B.Cu")
+		(start 178 108.15)
+		(end 178 68)
+		(width 1)
+		(layer "F.Cu")
 		(net 6)
 	)
 	(segment
-		(start 158 51)
-		(end 151 58)
-		(width 2)
-		(layer "B.Cu")
+		(start 75 78)
+		(end 84.01 68.99)
+		(width 1)
+		(layer "F.Cu")
 		(net 6)
 	)
 	(segment
-		(start 151 79)
-		(end 146 84)
-		(width 2)
-		(layer "B.Cu")
+		(start 84.01 68.99)
+		(end 84.01 55.5)
+		(width 1)
+		(layer "F.Cu")
 		(net 6)
 	)
 	(segment
-		(start 175.701 62.701)
-		(end 164 51)
-		(width 2)
-		(layer "B.Cu")
+		(start 101.7 55.5)
+		(end 84.01 55.5)
+		(width 1)
+		(layer "F.Cu")
 		(net 6)
 	)
 	(segment
-		(start 135.11 84)
-		(end 124.65 73.54)
-		(width 2)
-		(layer "B.Cu")
+		(start 105.95 59.75)
+		(end 105.95 50.75)
+		(width 1)
+		(layer "F.Cu")
 		(net 6)
 	)
@@
 	)
 	(segment
+		(start 84 129.4)
+		(end 74.559 119.959)
+		(width 4)
+		(layer "B.Cu")
+		(net 7)
+	)
+	(segment
 		(start 76.39 71.896948)
 		(end 76.39 55.5)
@@
 	)
 	(segment
-		(start 32 82)
-		(end 27 87)
+		(start 74.559 119.959)
+		(end 64.9 119.959)
 		(width 4)
 		(layer "B.Cu")
@@
 	)
 	(segment
-		(start 80.1 125.5)
-		(end 84 129.4)
-		(width 1)
+		(start 32 82)
+		(end 27 87)
+		(width 4)
 		(layer "B.Cu")
 		(net 7)
@@
 		(layer "B.Cu")
 		(net 7)
-	)
-	(segment
-		(start 64.9 125.5)
-		(end 80.1 125.5)
-		(width 1)
-		(layer "B.Cu")
-		(net 7)
